File: eagle/projekt/president_george/adapterplatine.brd (EAGLE design)
At the start: 60 x 60 mm, 28 parts, among them IC1 MAX232ECWE, U1 52207-1085

Commit message: - checking the brd files
Routing:
- net VCC: track 113.9 -> 100.8 mm
- net N$12: track 89.4 -> 81.1 mm
- net N$9: track 56.0 -> 61.7 mm
- net GND: track 232.5 -> 229.5 mm
- net N$14: track 33.1 -> 31.2 mm, vias 0 -> 1
- net N$10: track 51.6 -> 53.4 mm
- net N$2: track 25.3 -> 24.3 mm
- net N$3: track 6.37 -> 5.76 mm, vias 2 -> 0
- net N$11: vias 1 -> 0
